File: PCB/PCB_V1/PCB_V1.kicad_sch (KiCad schematic)
At the start: 18 parts, among them J1 Conn_01x10, J2 Conn_01x03, U1 STM32G431KBTx, U2 MCP6002-xSN, U3 BU33SD5WG-TR

Commit message: V1.1
Parts:
- renumbered J1 to J1_Afficheur
Connections:
- net LED0: now also U1.5 (PA0)
- net LED1: now also U1.6 (PA1)
- net LED2: now also U1.7 (PA2)
- net LED3: now also U1.8 (PA3)
- net LED4: now also U1.9 (PA4)
- net LED5: now also U1.10 (PA5)
- net LED6: now also U1.11 (PA6)
- net LED7: now also U1.12 (PA7)
- net LED_COM0: now also U1.24 (PA14)
- net LED_COM1: now also U1.25 (PA15)
- net Output_Pedale: now also U1.18 (PA8)
- net USART_TX: now reaches U1.19 (PA9)
Other:
- moved on the sheet: C1, U2B, U2C

Commit message: +2 gros boutons
Parts:
- added J1: Conn_01x03, symbol Connector_Generic:Conn_01x03
- added R7, R8: R, symbol Device:R
Connections:
- net GND: now also J1.3 (Pin_3)
- net SW_UP: now reaches U1.13 (PB0)
- net SW_UP: now also J1.1 (Pin_1), R7.2
- net SW_DOWN: now reaches U1.26 (PB3)
- net SW_DOWN: now also J1.2 (Pin_2), R8.2
- new net +3.3VD: R7.1, R8.1
