File: Hardware/PCB/PCB_V1/PCB_V1.kicad_pcb (KiCad board)
At the start: 2 copper layers, 70 x 92 mm, 39 parts, among them J1 Conn_01x03, J2 Conn_01x03, J3 Conn_ST_STDC14, J4 Conn_01x02, J5 Conn_01x02, J7 Conn_01x07, J8_afficheur1 Conn_01x10, Q1 DTA123J, Q2 DTA123J, U1 STM32G431KBTx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

Commit message: pcb complet
Parts:
- removed H6: MountingHole_Pad, MountingHole:MountingHole_4mm_Pad_TopBottom
- added D1: LED, LED_SMD:LED_0603_1608Metric, F.Cu at (68.0, 73.8)
- added D2: LED, LED_SMD:LED_0603_1608Metric, F.Cu at (68.1, 77.7)
- added J8: PRT-09536, PRT-09536:PRT09536, F.Cu at (100.5, 58.0)
- added JP1: SolderJumper1, Jumper:SolderJumper-2_P1.3mm_Open_TrianglePad1.0x1.5mm, F.Cu at (95.5, 68.0)
- added JP2: SolderJumper, Jumper:SolderJumper-2_P1.3mm_Open_TrianglePad1.0x1.5mm, F.Cu at (99.0, 68.0)
- added R1: 1000, Resistor_SMD:R_0402_1005Metric, F.Cu at (67.7, 75.5)
- added R11: 1000, Resistor_SMD:R_0402_1005Metric, F.Cu at (67.8, 79.5)
- moved R6 132.8 mm to (63.2, 119.9)
- moved R5 131.7 mm to (65.2, 120.2), turned to -90 degrees
- moved R3 130.5 mm to (63.2, 121.2)
- moved R4 126.0 mm to (66.9, 120.2), turned to 90 degrees
- moved J1 124.0 mm to (116.0, 119.0), turned to 90 degrees
- moved R2 122.6 mm to (73.0, 122.5), turned to 180 degrees
- moved J5 119.6 mm to (69.0, 58.8), turned to 180 degrees
- moved J4 100.1 mm to (79.0, 58.8), turned to 180 degrees
- moved R10 96.0 mm to (95.5, 71.3), turned to -90 degrees
- moved R8 94.0 mm to (109.0, 119.0), turned to 180 degrees
- moved R9 92.4 mm to (99.0, 71.3), turned to 90 degrees
- moved R7 88.4 mm to (109.0, 116.5), turned to 180 degrees
- moved J8_afficheur1 81.6 mm to (116.0, 106.5), turned to 90 degrees
- moved RV1 57.1 mm to (73.0, 119.0), turned to -90 degrees
- moved Q2 39.6 mm to (74.1, 76.3)
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Connections:
- Q1 pad 2: +3V3 -> +3.3V
- Q2 pad 2: +3V3 -> +3.3V
- R10 pad 1: +5V -> Net-(JP1-B)
- R10 pad 2: Net-(J6-Pad4) -> +5V
- U1 pad 31: unconnected-(U1-PB8-Pad31) -> Net-(D2-A)
Routing:
- net LED_COM0: track 0.00 -> 94.5 mm, vias 0 -> 2
- net LED_COM1: track 0.00 -> 94.0 mm, vias 0 -> 2
- net LED0_SEG: track 0.00 -> 73.5 mm
- net USART_TX: track 0.00 -> 69.6 mm, vias 0 -> 2
- net LED1_SEG: track 0.00 -> 67.8 mm
- net LED2_SEG: track 0.00 -> 64.9 mm
- net LED3_SEG: track 0.00 -> 63.6 mm
- net LED4_SEG: track 0.00 -> 62.1 mm
- net LED7_SEG: track 0.00 -> 60.9 mm, vias 0 -> 1
- net LED5_SEG: track 0.00 -> 60.5 mm
- net SW_UP: track 0.00 -> 57.9 mm, vias 0 -> 2
- net LED9: track 0.00 -> 56.9 mm, vias 0 -> 1
- net LED11: track 0.00 -> 56.8 mm, vias 0 -> 1
- net LED10: track 0.00 -> 56.7 mm, vias 0 -> 1
- net LED12: track 0.00 -> 55.6 mm, vias 0 -> 1
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- added copper zone on In2.Cu, net +3.3V
- added copper zone on In2.Cu, net +3.3VA
- added copper zone on B.Cu, net GND
- added copper zone on F.Cu, net GND
- added copper zone on In1.Cu, net GND
Other:
- board size 70 x 92 mm -> 78 x 92 mm
- copper layers 2 -> 4

Commit message: gerber 2
Other:
- board text added: "Alexian PREVOST Iprahim TURGUT Sacha CHERIFI V 1.0.0.0.0.1"
Changed lines of the file:
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@@
 		(tags "SOT TO_SOT_SMD")
 		(property "Reference" "Q2"
-			(at 3.1125 -1.1 360)
+			(at 3.1125 -1.1 0)
 			(layer "F.SilkS")
 			(effects
@@
 		)
 		(property "Value" "DTA123J"
-			(at 0 2.4 360)
+			(at 0 2.4 0)
 			(layer "F.Fab")
 			(effects
@@
 		)
 		(property "Footprint" "Package_TO_SOT_SMD:SOT-23-3"
-			(at 0 0 360)
+			(at 0 0 0)
 			(layer "F.Fab")
 			(hide yes)
@@
 		)
 		(property "Datasheet" ""
-			(at 0 0 360)
+			(at 0 0 0)
 			(layer "F.Fab")
 			(hide yes)
@@
 		)
 		(property "Description" "Digital PNP Transistor, 2k2/47k, SOT-23"
-			(at 0 0 360)
+			(at 0 0 0)
 			(layer "F.Fab")
 			(hide yes)
@@
 		)
 		(fp_text user "${REFERENCE}"
-			(at 0 0 360)
+			(at 0 0 0)
 			(layer "F.Fab")
 			(effects
@@
 		)
 		(property "Value" "330"
-			(at 0 1.17 360)
+			(at 0 1.17 0)
 			(layer "F.Fab")
 			(effects
@@
 		)
 		(fp_text user "${REFERENCE}"
-			(at 0 0 360)
+			(at 0 0 0)
 			(layer "F.Fab")
 			(effects
@@
 		(tags "SOT TO_SOT_SMD")
 		(property "Reference" "U3"
-			(at 0.6 2.6 360)
+			(at 0.6 2.6 0)
 			(layer "F.SilkS")
 			(effects
@@
 		)
 		(property "Value" "BU33SD5WG-TR"
-			(at 0 2.4 360)
+			(at 0 2.4 0)
 			(layer "F.Fab")
 			(effects
@@
 		)
 		(property "Footprint" "Package_TO_SOT_SMD:SOT-23-5"
-			(at 0 0 360)
+			(at 0 0 0)
 			(layer "F.Fab")
 			(hide yes)
@@
 		)
 		(property "Datasheet" "http://ww1.microchip.com/downloads/en/DeviceDoc/22053C.pdf"
-			(at 0 0 360)
+			(at 0 0 0)
 			(layer "F.Fab")
 			(hide yes)
@@
 		)
 		(property "Description" "150mA, Tiny CMOS LDO With Shutdown, Fixed Voltage, SOT-23-5"
-			(at 0 0 360)
+			(at 0 0 0)
 			(layer "F.Fab")
 			(hide yes)
@@
 		)
 		(fp_text user "${REFERENCE}"
-			(at 0 0 360)
+			(at 0 0 0)
 			(layer "F.Fab")
 			(effects
@@
 		(tags "connector JST XH vertical")
 		(property "Reference" "J4"
-			(at 0.9 4.75 360)
+			(at 0.9 4.75 0)
 			(layer "F.SilkS")
 			(effects
@@
 		)
 		(property "Value" "Conn_01x02"
-			(at 1.25 4.6 360)
+			(at 1.25 4.6 0)
 			(layer "F.Fab")
 			(effects
@@
 		)
 		(fp_text user "${REFERENCE}"
-			(at 1.25 2.7 360)
+			(at 1.25 2.7 0)
 			(layer "F.Fab")
 			(effects
@@
 		(tags "capacitor")
 		(property "Reference" "C1"
-			(at 0 -1.16 360)
+			(at 0 -1.16 0)
 			(layer "F.SilkS")
 			(effects
@@
 		)
 		(property "Value" "100nF"
-			(at 0 1.16 360)
+			(at 0 1.16 0)
 			(layer "F.Fab")
 			(effects
@@
 		)
 		(fp_text user "${REFERENCE}"
-			(at 0 0 360)
+			(at 0 0 0)
 			(layer "F.Fab")
 			(effects
@@
 		(tags "resistor")
 		(property "Reference" "R3"
-			(at -2.2 0.2 360)
+			(at -2.2 0.2 0)
 			(layer "F.SilkS")
 			(effects
@@
 		)
 		(property "Value" "110k"
-			(at 0 1.17 360)
+			(at 0 1.17 0)
 			(layer "F.Fab")
 			(effects
@@
 		)
 		(fp_text user "${REFERENCE}"
-			(at 0 0 360)
+			(at 0 0 0)
 			(layer "F.Fab")
 			(effects
@@
 		(tags "resistor")
 		(property "Reference" "R6"
-			(at -2.205 0 360)
+			(at -2.205 0 0)
 			(layer "F.SilkS")
 			(effects
@@
 		)
 		(property "Value" "110k"
-			(at 0 1.17 360)
+			(at 0 1.17 0)
 			(layer "F.Fab")
 			(effects
@@
 		)
 		(fp_text user "${REFERENCE}"
-			(at 0 0 360)
+			(at 0 0 0)
 			(layer "F.Fab")
 			(effects
@@
 		(tags "inductor")
 		(property "Reference" "L1"
-			(at 2.475 0.01 360)
+			(at 2.475 0.01 0)
 			(layer "F.SilkS")
 			(effects
@@
 		)
 		(property "Value" "39n"
-			(at 0 1.43 360)
+			(at 0 1.43 0)
 			(layer "F.Fab")
 			(effects
@@
 		)
 		(fp_text user "${REFERENCE}"
-			(at 0 0 360)
+			(at 0 0 0)
 			(layer "F.Fab")
 			(effects
@@
 		(tags "SOT TO_SOT_SMD")
 		(property "Reference" "Q1"
-			(at 3.1125 -1.05 360)
+			(at 3.1125 -1.05 0)
 			(layer "F.SilkS")
 			(effects
@@
 		)
 		(property "Value" "DTA123J"
-			(at 0 2.4 360)
+			(at 0 2.4 0)
 			(layer "F.Fab")
 			(effects
@@
 		)
 		(property "Footprint" "Package_TO_SOT_SMD:SOT-23-3"
-			(at 0 0 360)
+			(at 0 0 0)
 			(layer "F.Fab")
 			(hide yes)
@@
 		)
 		(property "Datasheet" ""
-			(at 0 0 360)
+			(at 0 0 0)
 			(layer "F.Fab")
 			(hide yes)
@@
 		)
 		(property "Description" "Digital PNP Transistor, 2k2/47k, SOT-23"
-			(at 0 0 360)
+			(at 0 0 0)
 			(layer "F.Fab")
 			(hide yes)
@@
 		)
 		(fp_text user "${REFERENCE}"
-			(at 0 0 360)
+			(at 0 0 0)
 			(layer "F.Fab")
 			(effects
@@
 		(tags "resistor")
 		(property "Reference" "R8"
-			(at 2.4 0 360)
+			(at 2.4 0 0)
 			(layer "F.SilkS")
 			(effects
@@
 		)
 		(property "Value" "47k"
-			(at 0 1.17 360)
+			(at 0 1.17 0)
 			(layer "F.Fab")
 			(effects
@@
 		)
 		(fp_text user "${REFERENCE}"
-			(at 0 0 360)
+			(at 0 0 0)
 			(layer "F.Fab")
 			(effects
@@
 		(tags "resistor")
 		(property "Reference" "R7"
-			(at 2.2 -0.1 360)
+			(at 2.2 -0.1 0)
 			(layer "F.SilkS")
 			(effects
@@
 		)
 		(property "Value" "47k"
-			(at 0 1.17 360)
+			(at 0 1.17 0)
 			(layer "F.Fab")
 			(effects
@@
 		)
 		(fp_text user "${REFERENCE}"
-			(at 0 0 360)
+			(at 0 0 0)
 			(layer "F.Fab")
 			(effects
@@
 		(tags "resistor")
 		(property "Reference" "R11"
-			(at 2.7025 0 360)
+			(at 2.7025 0 0)
 			(layer "F.SilkS")
 			(effects
@@
 		)
 		(property "Value" "1000"
-			(at 0 1.17 360)
+			(at 0 1.17 0)
 			(layer "F.Fab")
 			(effects
@@
 		)
 		(fp_text user "${REFERENCE}"
-			(at 0 0 360)
+			(at 0 0 0)
 			(layer "F.Fab")
 			(effects
@@
 		(tags "connector JST XH vertical")
 		(property "Reference" "J5"
-			(at 1.2 4.65 360)
+			(at 1.2 4.65 0)
 			(layer "F.SilkS")
 			(effects
@@
 		)
 		(property "Value" "Conn_01x02"
-			(at 1.25 4.6 360)
+			(at 1.25 4.6 0)
 			(layer "F.Fab")
 			(effects
@@
 		)
 		(fp_text user "${REFERENCE}"
-			(at 1.25 2.7 360)
+			(at 1.25 2.7 0)
 			(layer "F.Fab")
 			(effects
@@
 		(tags "resistor")
 		(property "Reference" "R1"
-			(at 2.49 0 360)
+			(at 2.49 0 0)
 			(layer "F.SilkS")
 			(effects
@@
 		)
 		(property "Value" "1000"
-			(at 0 1.17 360)
+			(at 0 1.17 0)
 			(layer "F.Fab")
 			(effects
@@
 		)
 		(fp_text user "${REFERENCE}"
-			(at 0 0 360)
+			(at 0 0 0)
 			(layer "F.Fab")
 			(effects
@@
 		(tags "connector JST XH vertical")
 		(property "Reference" "J7"
-			(at 7.5 -3.55 360)
+			(at 7.5 -3.55 0)
 			(layer "F.SilkS")
 			(effects
@@
 		)
 		(property "Value" "Conn_01x07"
-			(at 7.5 4.6 360)
+			(at 7.5 4.6 0)
 			(layer "F.Fab")
 			(effects
@@
 		)
 		(fp_text user "${REFERENCE}"
-			(at 7.5 2.7 360)
+			(at 7.5 2.7 0)
 			(layer "F.Fab")
 			(effects
@@
 		(tags "Surface mounted pin header SMD 2x07 1.27mm double row")
 		(property "Reference" "J3"
-			(at -0.025 5.94 360)
+			(at -0.025 5.94 0)
 			(layer "F.SilkS")
 			(effects
@@
 		)
 		(property "Value" "Conn_ST_STDC14"
-			(at 0 5.505 360)
+			(at 0 5.505 0)
 			(layer "F.Fab")
 			(effects
@@
 		(tags "connector JST XH vertical")
 		(property "Reference" "J2"
-			(at 2.5 4.5 360)
+			(at 2.5 4.5 0)
 			(layer "F.SilkS")
 			(effects
@@
 		)
 		(property "Value" "Conn_01x03"
-			(at 2.5 4.6 360)
+			(at 2.5 4.6 0)
 			(layer "F.Fab")
 			(effects
@@
 		)
 		(fp_text user "${REFERENCE}"
-			(at 2.5 2.7 360)
+			(at 2.5 2.7 0)
 			(layer "F.Fab")
 			(effects
@@
 		(layer "Edge.Cuts")
 	)
+	(gr_text "Alexian PREVOST\nIprahim TURGUT\nSacha CHERIFI\nV 1.0.0.0.0.1"
+		(at 62.6 116.2 0)
+		(layer "B.SilkS")
+		(effects
+			(font
+				(size 1 1)
+				(thickness 0.1)
+			)
+			(justify left bottom mirror)
+		)
+	)
 	(dimension
 		(type aligned)
@@
 	)
 	(segment
-		(start 64 95)
-		(end 83 114)
+		(start 64 86.5)
+		(end 64 96.8)
 		(width 0.3)
 		(layer "B.Cu")
@@
 	)
 	(segment
-		(start 83 114)
-		(end 83 131)
+		(start 63.85 86.35)
+		(end 64 86.5)
 		(width 0.3)
 		(layer "B.Cu")
@@
 	)
 	(segment
-		(start 64 86.5)
-		(end 64 95)
+		(start 83 115.8)
+		(end 83 131)
 		(width 0.3)
 		(layer "B.Cu")
@@
 	)
 	(segment
-		(start 63.85 86.35)
-		(end 64 86.5)
+		(start 64 96.8)
+		(end 83 115.8)
 		(width 0.3)
 		(layer "B.Cu")
